File: pcb/v2/ESP-DubSiren-V2.kicad_sch (KiCad schematic)
At the start: 49 parts, among them J1 USB4085-GF-A, J2 RCJ-2123, SW5 RESET, SW6 BOOT, U1 ESP32-S3-WROOM-1U-N16R8, U2 MPM3612GLQ-33-Z, U3 74HC4051D, U4 USBLC6-2SC6, U5 Adafruit 5393, U6 Adafruit 6250

Commit message: pcb-v2: add validated Bourns controls and USB input slew stage
Parts:
- added C10: 1u, Capacitor_SMD:C_0603_1608Metric, symbol Device:C
- added C11: 10n C0G 50V, Capacitor_SMD:C_0603_1608Metric, symbol Device:C
- added RV1, RV2, RV3, RV4, RV5, RV6: 20k PTV111-3420A-B203, ESP-DubSiren-V2-Mechanical:Bourns_PTV111-3, symbol Device:R_Potentiometer
- added RV7: 10k PTV111-1420A-B103, ESP-DubSiren-V2-Mechanical:Bourns_PTV111-1, symbol Device:R_Potentiometer
- added SW7: PEC11R-4120F-S0018, ESP-DubSiren-V2-Mechanical:Bourns_PEC11R-4120F-S0018, symbol Device:RotaryEncoder_Switch
- added U7: TPS22918DBVR, Package_TO_SOT_SMD:SOT-23-6, symbol ESP-DubSiren-V2:TPS22918DBVR
Connections:
- net +5V: now also U7.6 (VOUT); no longer D1.1 (K), F1.2
- net ENC_A: now also SW7.A
- net ENC_B: now also SW7.B
- net ENC_SW: now also SW7.S1
- net GND: now also C10.2, C11.2, RV1.1, RV2.1, RV3.1, RV4.1, RV5.1, RV6.1, RV7.1, SW7.C, SW7.S2, U7.2 (GND)
- net MASTER: now also RV7.2
- net POT1: now also RV1.2
- net POT1_TOP: now also RV1.3
- net POT2: now also RV2.2
- net POT2_TOP: now also RV2.3
- net POT3: now also RV3.2
- net POT3_TOP: now also RV3.3
- net POT4: now also RV4.2
- net POT4_TOP: now also RV4.3
- net POT5: now also RV5.2
- net POT5_TOP: now also RV5.3
- net POT6: now also RV6.2
- net POT6_TOP: now also RV6.3
- net POT7_TOP: now also RV7.3
- new net VBUS_PROTECTED: C10.1, D1.1 (K), F1.2, U7.1 (VIN), U7.3 (ON)
- new net VBUS_SLEW_CT: C11.1, U7.4 (CT)
- no-connect marks 26 -> 27

Commit message: pcb-v2: complete schematic with verified native CHERRY footprints
Parts:
- added SW1, SW2, SW3, SW4: MX2A-11NW, Button_Switch_Keyboard:SW_Cherry_MX_1.00u_PCB, symbol Switch:SW_SPST
Connections:
- net BTN1: now also SW1.1 (A)
- net BTN2: now also SW2.1 (A)
- net BTN3: now also SW3.1 (A)
- net BTN4: now also SW4.1 (A)
- net GND: now also SW1.2 (B), SW2.2 (B), SW3.2 (B), SW4.2 (B)
Other:
- note added: "PROTOTYPE - all controls populated; USB power policy and bench qualification pending"
- note removed: "DRAFT - pending mechanical pin-map acceptance and USB inrush review"
