File: pcb/v2/ESP-DubSiren-V2.kicad_pcb (KiCad board)
At the start: 2 copper layers, 0 parts

Commit message: pcb-v2: save routed and mechanical checkpoint at requested stop
Parts:
- added C1: 22u, Capacitor_SMD:C_0805_2012Metric, B.Cu at (14.5, 31.1)
- added C10: 1u, Capacitor_SMD:C_0603_1608Metric, B.Cu at (19.5, 22.9)
- added C11: 10n C0G 50V, Capacitor_SMD:C_0603_1608Metric, B.Cu at (28.0, 21.1)
- added C2: 100n, Capacitor_SMD:C_0603_1608Metric, B.Cu at (15.5, 33.2)
- added C3: 22u, Capacitor_SMD:C_0805_2012Metric, B.Cu at (17.0, 27.0)
- added C4: 100n, Capacitor_SMD:C_0603_1608Metric, B.Cu at (17.0, 24.7)
- added C5: 22u, Capacitor_SMD:C_0805_2012Metric, B.Cu at (20.5, 59.0)
- added C6: 100n, Capacitor_SMD:C_0603_1608Metric, B.Cu at (24.0, 56.1)
- added C7: 1u, Capacitor_SMD:C_0603_1608Metric, B.Cu at (23.5, 50.5)
- added C8: 100n, Capacitor_SMD:C_0603_1608Metric, B.Cu at (31.5, 73.4)
- added C9: 100n, Capacitor_SMD:C_0603_1608Metric, B.Cu at (24.0, 53.6)
- added D1: SMF5.0A, Diode_SMD:D_SOD-123F, B.Cu at (34.0, 22.5)
- added F1: 1.1A PTC, ESP-DubSiren-V2-Electrical:Bel_0ZCG0110CF2B_1812, B.Cu at (34.5, 18.0)
- added H1: MountingHole_3.2mm_M3, MountingHole:MountingHole_3.2mm_M3, F.Cu at (12.0, 12.0)
- added H2: MountingHole_3.2mm_M3, MountingHole:MountingHole_3.2mm_M3, F.Cu at (113.0, 12.0)
- added H3: MountingHole_3.2mm_M3, MountingHole:MountingHole_3.2mm_M3, F.Cu at (12.0, 128.0)
- added H4: MountingHole_3.2mm_M3, MountingHole:MountingHole_3.2mm_M3, F.Cu at (113.0, 128.0)
- added J1: USB4085-GF-A, Connector_USB:USB_C_Receptacle_GCT_USB4085, B.Cu at (42.0, 10.0)
- added J2: RCJ-2123, ESP-DubSiren-V2-Mechanical:SameSky_RCJ-2123, B.Cu at (92.5, 12.0)
- added R1: 10, Resistor_SMD:R_0603_1608Metric, B.Cu at (21.5, 28.2)
- added R10: 4.7k, Resistor_SMD:R_0603_1608Metric, B.Cu at (98.8, 33.0)
- added R11: 4.7k, Resistor_SMD:R_0603_1608Metric, B.Cu at (28.8, 108.0)
- added R12: 4.7k, Resistor_SMD:R_0603_1608Metric, B.Cu at (63.8, 108.0)
- added R13: 4.7k, Resistor_SMD:R_0603_1608Metric, B.Cu at (98.8, 108.0)
- added R14: 4.7k, Resistor_SMD:R_0603_1608Metric, B.Cu at (17.0, 20.0)
- added R15: 10k, Resistor_SMD:R_0603_1608Metric, B.Cu at (52.0, 44.0)
- added R16: 10k, Resistor_SMD:R_0603_1608Metric, B.Cu at (52.0, 46.0)
- added R17: 10k, Resistor_SMD:R_0603_1608Metric, B.Cu at (52.0, 50.0)
- added R18: 10k, Resistor_SMD:R_0603_1608Metric, B.Cu at (52.0, 52.0)
- added R19: 10k, Resistor_SMD:R_0603_1608Metric, B.Cu at (52.0, 58.0)
- added R2: 22, Resistor_SMD:R_0603_1608Metric, B.Cu at (24.0, 42.4)
- added R20: 10k, Resistor_SMD:R_0603_1608Metric, B.Cu at (52.0, 56.0)
- added R21: 10k, Resistor_SMD:R_0603_1608Metric, B.Cu at (52.0, 54.0)
- added R3: 22, Resistor_SMD:R_0603_1608Metric, B.Cu at (24.0, 40.6)
- added R4: 5.1k, Resistor_SMD:R_0603_1608Metric, B.Cu at (52.0, 10.5)
- added R5: 5.1k, Resistor_SMD:R_0603_1608Metric, B.Cu at (52.0, 14.5)
- added R6: 10k, Resistor_SMD:R_0603_1608Metric, B.Cu at (20.5, 48.5)
- added R7: 10k, Resistor_SMD:R_0603_1608Metric, B.Cu at (49.0, 39.0)
- added R8: 4.7k, Resistor_SMD:R_0603_1608Metric, B.Cu at (30.5, 35.0)
- added R9: 4.7k, Resistor_SMD:R_0603_1608Metric, B.Cu at (65.5, 32.0)
- added RV1: 20k PTV111-3420A-B203, ESP-DubSiren-V2-Mechanical:Bourns_PTV111-3, F.Cu at (27.5, 26.0)
- added RV2: 20k PTV111-3420A-B203, ESP-DubSiren-V2-Mechanical:Bourns_PTV111-3, F.Cu at (62.5, 26.0)
- added RV3: 20k PTV111-3420A-B203, ESP-DubSiren-V2-Mechanical:Bourns_PTV111-3, F.Cu at (97.5, 26.0)
- added RV4: 20k PTV111-3420A-B203, ESP-DubSiren-V2-Mechanical:Bourns_PTV111-3, F.Cu at (27.5, 94.0)
- added RV5: 20k PTV111-3420A-B203, ESP-DubSiren-V2-Mechanical:Bourns_PTV111-3, F.Cu at (62.5, 94.0)
- added RV6: 20k PTV111-3420A-B203, ESP-DubSiren-V2-Mechanical:Bourns_PTV111-3, F.Cu at (97.5, 94.0)
- added RV7: 10k PTV111-1420A-B103, ESP-DubSiren-V2-Mechanical:Bourns_PTV111-1, B.Cu at (23.0, 9.50)
- added SW1: MX2A-11NW, Button_Switch_Keyboard:SW_Cherry_MX_1.00u_PCB, F.Cu at (30.0, 116.9)
- added SW2: MX2A-11NW, Button_Switch_Keyboard:SW_Cherry_MX_1.00u_PCB, F.Cu at (53.3, 116.9)
- added SW3: MX2A-11NW, Button_Switch_Keyboard:SW_Cherry_MX_1.00u_PCB, F.Cu at (76.7, 116.9)
- added SW4: MX2A-11NW, Button_Switch_Keyboard:SW_Cherry_MX_1.00u_PCB, F.Cu at (100.0, 116.9)
- added SW5: RESET, ESP-DubSiren-V2-Electrical:CK_PTS636SM43SMTR_LFS, B.Cu at (12.0, 58.0)
- added SW6: BOOT, ESP-DubSiren-V2-Electrical:CK_PTS636SM43SMTR_LFS, B.Cu at (12.0, 73.0)
- added SW7: PEC11R-4120F-S0018, ESP-DubSiren-V2-Mechanical:Bourns_PEC11R-4120F-S0018, F.Cu at (97.5, 60.0)
- added TP1: +5V, TestPoint:TestPoint_Pad_D1.0mm, B.Cu at (32.0, 25.0)
- added TP2: +3V3, TestPoint:TestPoint_Pad_D1.0mm, B.Cu at (13.0, 37.0)
- added TP3: GND, TestPoint:TestPoint_Pad_D1.0mm, B.Cu at (12.0, 84.0)
- added TP4: ADC_MUX, TestPoint:TestPoint_Pad_D1.0mm, B.Cu at (24.5, 60.0)
- added TP5: AUDIO_MONO, TestPoint:TestPoint_Pad_D1.0mm, B.Cu at (92.5, 30.0)
- added TP6: UART_TX, TestPoint:TestPoint_Pad_D1.0mm, B.Cu at (47.0, 60.0)
- added TP7: UART_RX, TestPoint:TestPoint_Pad_D1.0mm, B.Cu at (50.0, 60.0)
- added U1: ESP32-S3-WROOM-1U-N16R8, ESP-DubSiren-V2-Electrical:Espressif_ESP32-S3-WROOM-1U, B.Cu at (36.0, 49.0)
- added U2: MPM3612GLQ-33-Z, ESP-DubSiren-V2-Electrical:MPS_MPM3612GLQ-33_LGA-8-1EP_3x3mm, B.Cu at (18.0, 30.0)
- added U3: 74HC4051D, Package_SO:SOIC-16_3.9x9.9mm_P1.27mm, B.Cu at (26.0, 69.0)
- added U4: USBLC6-2SC6, Package_TO_SOT_SMD:SOT-23-6, B.Cu at (45.0, 15.0)
- added U5: Adafruit 5393, ESP-DubSiren-V2-Mechanical:Adafruit_5393_DisplayFace, F.Cu at (63.5, 60.0)
- added U6: Adafruit 6250, ESP-DubSiren-V2-Mechanical:Adafruit_6250_ComponentFace, B.Cu at (76.0, 48.5)
- added U7: TPS22918DBVR, Package_TO_SOT_SMD:SOT-23-6, B.Cu at (24.0, 22.0)
Routing:
- net +3V3: track 0.00 -> 334.7 mm, vias 0 -> 6
- net /BTN1: track 0.00 -> 110.0 mm, vias 0 -> 2
- net /BTN4: track 0.00 -> 103.5 mm, vias 0 -> 6
- net /BTN2: track 0.00 -> 102.2 mm, vias 0 -> 2
- net /POT6: track 0.00 -> 90.6 mm, vias 0 -> 2
- net /BTN3: track 0.00 -> 89.5 mm, vias 0 -> 4
- net /ENC_B: track 0.00 -> 85.1 mm, vias 0 -> 4
- net +5V: track 0.00 -> 85.0 mm, vias 0 -> 4
- net /POT3: track 0.00 -> 82.4 mm, vias 0 -> 6
- net /MASTER: track 0.00 -> 73.9 mm, vias 0 -> 2
- net /ENC_A: track 0.00 -> 65.8 mm, vias 0 -> 2
- net /BOOT: track 0.00 -> 62.6 mm, vias 0 -> 2
- net /POT2: track 0.00 -> 61.4 mm, vias 0 -> 4
- net /USB_DM_CONN: track 0.00 -> 59.5 mm
- net /TFT_LITE: track 0.00 -> 59.0 mm, vias 0 -> 2
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- added copper zone on B.Cu, net GND
- added copper zone on F.Cu, net GND
Other:
- board outline added: 113 x 130.5 mm
